File: Hardware/SmartHydroponics.sch (KiCad schematic (older format))
At the start: 62 parts, among them J1 Barrel_Jack, J10 A2501WR-2P1, J15 S2B-ZR, J2 Header_1x6, J3 S3B-ZR, J4 BNC, J7 A2501WR-2P1, J8 A2501WR-2P1, J9 A2501WR-2P1, Q10 IRLML6346TRPBF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

Commit message: I do not remember. Sorry. Forgot to push. Sincerely Past David.
Parts:
- C31, C33, C61: TME CL10A106MO8NQNC -> CL32B106KAJNNNE
- C51: TME (none) -> CL10B104KO8NNNC
- C62, C71: TME (none) -> CL10A105KA8NNNC
- J10, J7, J8, J9: TME NXW-02K, NXG-02, NXG-T -> NX2500-02SMR
- J3: TME (none) -> S3B-ZR
- J4: TME (none) -> 5-1634556-0
- R111, R112, R113: TME (none) -> WF06P-150R-5%
- R32: TME WF06P-10K-5% -> CQ0603-49K9-1%
- R33: TME WF06P-10K-5% -> SMD0603-16K
- U1: TME (none) -> ESP32-WROOM-32D
Changed lines of the file:
@@
 F 2 "MRS_Passives:C1210" H 2200 1000 50  0001 C CNN
 F 3 "" H 2225 1600 50  0001 C CNN
-F 4 "CL10A106MO8NQNC" H 2200 1500 50  0001 C CNN "TME"
+F 4 "CL32B106KAJNNNE" H 2200 1500 50  0001 C CNN "TME"
 	1    2200 1500
 	1    0    0    -1
@@
 F 2 "MRS_Passives:C1210" H 5150 1000 50  0001 C CNN
 F 3 "" H 5175 1600 50  0001 C CNN
-F 4 "CL10A106MO8NQNC" H 5150 1500 50  0001 C CNN "TME"
+F 4 "CL32B106KAJNNNE" H 5150 1500 50  0001 C CNN "TME"
 	1    5150 1500
 	1    0    0    -1
@@
 F 2 "MRS_Connectors:A2501WR-2P1" H 10600 4000 50  0001 C CNN
 F 3 "https://www.tme.eu/Document/cd32a27eaa56cbe24bba92418ea31066/A2501WR-XP.pdf" H 10600 3900 50  0001 C CNN
-F 4 "NXW-02K, NXG-02, NXG-T" H 10600 3800 50  0001 C CNN "TME"
+F 4 "NX2500-02SMR" H 10600 3800 50  0001 C CNN "TME"
 	1    10600 4250
 	1    0    0    -1
@@
 F 2 "MRS_Connectors:A2501WR-2P1" H 10600 650 50  0001 C CNN
 F 3 "https://www.tme.eu/Document/cd32a27eaa56cbe24bba92418ea31066/A2501WR-XP.pdf" H 10600 550 50  0001 C CNN
-F 4 "NXW-02K, NXG-02, NXG-T" H 10600 450 50  0001 C CNN "TME"
+F 4 "NX2500-02SMR" H 10600 450 50  0001 C CNN "TME"
 	1    10600 900
 	1    0    0    -1
@@
 F 2 "MRS_Connectors:A2501WR-2P1" H 10600 1750 50  0001 C CNN
 F 3 "https://www.tme.eu/Document/cd32a27eaa56cbe24bba92418ea31066/A2501WR-XP.pdf" H 10600 1650 50  0001 C CNN
-F 4 "NXW-02K, NXG-02, NXG-T" H 10600 1550 50  0001 C CNN "TME"
+F 4 "NX2500-02SMR" H 10600 1550 50  0001 C CNN "TME"
 	1    10600 2000
 	1    0    0    -1
@@
 F 2 "MRS_Connectors:A2501WR-2P1" H 10600 2850 50  0001 C CNN
 F 3 "https://www.tme.eu/Document/cd32a27eaa56cbe24bba92418ea31066/A2501WR-XP.pdf" H 10600 2750 50  0001 C CNN
-F 4 "NXW-02K, NXG-02, NXG-T" H 10600 2650 50  0001 C CNN "TME"
+F 4 "NX2500-02SMR" H 10600 2650 50  0001 C CNN "TME"
 	1    10600 3100
 	1    0    0    -1
@@
 F 2 "MRS_Communication:ESP32-WROOM" H 2650 4700 50  0001 C CNN
 F 3 "https://www.espressif.com/sites/default/files/documentation/esp32-wroom-32_datasheet_en.pdf" H 2650 4600 50  0001 C CNN
+F 4 "ESP32-WROOM-32D" H 0   0   50  0001 C CNN "TME"
 	1    2650 5800
 	1    0    0    -1
@@
 F 2 "MRS_Passives:R0603" V 5150 1350 50  0001 C CNN
 F 3 "" V 4830 1350 50  0001 C CNN
-F 4 "WF06P-10K-5%" H 4750 1350 50  0001 C CNN "TME"
+F 4 "CQ0603-49K9-1%" H 4750 1350 50  0001 C CNN "TME"
 	1    4750 1350
 	1    0    0    -1
@@
 F 2 "MRS_Passives:R0603" V 5150 1650 50  0001 C CNN
 F 3 "" V 4830 1650 50  0001 C CNN
-F 4 "WF06P-10K-5%" H 4750 1650 50  0001 C CNN "TME"
+F 4 "SMD0603-16K" H 4750 1650 50  0001 C CNN "TME"
 	1    4750 1650
 	1    0    0    -1
@@
 F 2 "MRS_Passives:R0603" V 6300 6950 50  0001 C CNN
 F 3 "" V 5980 6950 50  0001 C CNN
+F 4 "WF06P-150R-5%" H 0   0   50  0001 C CNN "TME"
 	1    5900 6950
 	0    1    1    0
@@
 F 2 "MRS_Passives:R0603" V 6300 7350 50  0001 C CNN
 F 3 "" V 5980 7350 50  0001 C CNN
+F 4 "WF06P-150R-5%" H 0   0   50  0001 C CNN "TME"
 	1    5900 7350
 	0    1    1    0
@@
 F 2 "MRS_Passives:R0603" V 6300 7150 50  0001 C CNN
 F 3 "" V 5980 7150 50  0001 C CNN
+F 4 "WF06P-150R-5%" H 0   0   50  0001 C CNN "TME"
 	1    5900 7150
 	0    1    1    0
@@
 F 1 "BNC" H 4300 3900 50  0000 C CNN
 F 2 "MRS_Connectors:TE_BNC" H 4150 3950 50  0001 C CNN
-F 3 " ~" H 4150 3950 50  0001 C CNN
+F 3 "https://www.tme.eu/Document/61927071f94eba40dec04ddd7cae8ab1/5-1634556-0.pdf" H 4150 3950 50  0001 C CNN
+F 4 "5-1634556-0" H 0   0   50  0001 C CNN "TME"
 	1    4150 3950
 	-1   0    0    -1
@@
 F 2 "MRS_Passives:C0603" H 7550 2500 50  0001 C CNN
 F 3 "" H 7575 3100 50  0001 C CNN
+F 4 "CL10A105KA8NNNC" H 0   0   50  0001 C CNN "TME"
 	1    7550 3000
 	1    0    0    -1
@@
 F 2 "MRS_Passives:C0603" H 6900 3600 50  0001 C CNN
 F 3 "" H 6925 4200 50  0001 C CNN
+F 4 "CL10A105KA8NNNC" H 0   0   50  0001 C CNN "TME"
 	1    6900 4100
 	1    0    0    -1
@@
 F 2 "MRS_Passives:C0603" H 4050 2450 50  0001 C CNN
 F 3 "" H 4075 3050 50  0001 C CNN
+F 4 "CL10B104KO8NNNC" H 0   0   50  0001 C CNN "TME"
 	1    4050 2950
 	1    0    0    -1
@@
 F 2 "MRS_Passives:C1210" H 7050 2500 50  0001 C CNN
 F 3 "" H 7075 3100 50  0001 C CNN
-F 4 "CL10A106MO8NQNC" H 7050 3000 50  0001 C CNN "TME"
+F 4 "CL32B106KAJNNNE" H 7050 3000 50  0001 C CNN "TME"
 	1    7050 3000
 	1    0    0    -1
@@
 F 2 "MRS_Connectors:S3B-ZR" H 1350 3000 50  0001 C CNN
 F 3 "" H 900 3000 50  0001 C CNN
+F 4 "S3B-ZR" H 0   0   50  0001 C CNN "TME"
 	1    1350 3300
 	-1   0    0    -1
